File: audio.kicad_sch (KiCad schematic)
At the start: 36 parts

Commit message: Add files via upload
Connections:
- net AF_OUT: now reaches R?.1
Changed lines of the file:
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@@
+    )
+  )
+  (global_label "AF_OUT" (shape input) (at 146.05 83.82 180) (fields_autoplaced)
+    (effects (font (size 1.27 1.27)) (justify right))
+    (property "Intersheet References" "${INTERSHEET_REFS}" (id 0) (at 136.8636 83.7406 0)
+      (effects (font (size 1.27 1.27)) (justify right) hide)
     )
   )

Commit message: RF part update
Parts:
- C15, C16, C17, C18, C19, C20, C21, C22, C23, C24, C25, C26, C28: renamed from C?; footprint pkl_dipol:C_0603 -> Capacitor_SMD:C_0402_1005Metric
- LS1: renamed from LS?; footprint (none) -> Connector_PinHeader_2.54mm:PinHeader_1x02_P2.54mm_Vertical
- R10, R11, R12, R13, R14, R15, R16, R17, R18, R19: renamed from R?; footprint pkl_dipol:R_0603 -> Resistor_SMD:R_0402_1005Metric
- gave numbers to parts that had none: 12
