File: interface.kicad_sch (KiCad schematic)
At the start: 8 parts

Commit message: Add files via upload
Parts:
- added J?: OLED, Connector_PinHeader_2.54mm:PinHeader_1x07_P2.54mm_Vertical, symbol Connector_Generic:Conn_01x07
- added J?: UART, Connector_PinHeader_2.54mm:PinHeader_1x03_P2.54mm_Vertical, symbol Connector_Generic:Conn_01x03
Connections:
- net GND: now also J?.3 (Pin_3), J?.6 (Pin_6)
- new net OLED_CS: J?.3 (Pin_3)
- new net OLED_DC: J?.2 (Pin_2)
- new net OLED_RST: J?.1 (Pin_1)
- new net OLED_SPI_MOSI: J?.5 (Pin_5)
- new net OLED_SPI_SCK: J?.4 (Pin_4)
- new net USART1_RX: J?.1 (Pin_1)
- new net USART1_TX: J?.2 (Pin_2)
- new net VDD: J?.7 (Pin_7)
Changed lines of the file:
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@@
+    (stroke (width 0) (type solid) (color 0 0 0 0))
+  )
+  (wire (pts (xy 130.81 93.98) (xy 135.89 93.98))
     (stroke (width 0) (type solid) (color 0 0 0 0))
   )
@@
     (stroke (width 0) (type solid) (color 0 0 0 0))
   )
+  (wire (pts (xy 82.55 96.52) (xy 85.09 96.52))
+    (stroke (width 0) (type solid) (color 0 0 0 0))
+  )
   (wire (pts (xy 204.47 90.17) (xy 208.28 90.17))
     (stroke (width 0) (type solid) (color 0 0 0 0))
@@
     (stroke (width 0) (type solid) (color 0 0 0 0))
   )
+  (wire (pts (xy 135.89 106.68) (xy 130.81 106.68))
+    (stroke (width 0) (type solid) (color 0 0 0 0))
+  )
   (wire (pts (xy 208.28 116.84) (xy 208.28 119.38))
     (stroke (width 0) (type solid) (color 0 0 0 0))
@@
     (stroke (width 0) (type solid) (color 0 0 0 0))
   )
+  (wire (pts (xy 135.89 109.22) (xy 133.35 109.22))
+    (stroke (width 0) (type solid) (color 0 0 0 0))
+  )
   (wire (pts (xy 208.28 107.95) (xy 208.28 116.84))
     (stroke (width 0) (type solid) (color 0 0 0 0))
   )
+  (wire (pts (xy 133.35 109.22) (xy 133.35 91.44))
+    (stroke (width 0) (type solid) (color 0 0 0 0))
+  )
+  (wire (pts (xy 82.55 93.98) (xy 85.09 93.98))
+    (stroke (width 0) (type solid) (color 0 0 0 0))
+  )
   (wire (pts (xy 208.28 90.17) (xy 208.28 99.06))
     (stroke (width 0) (type solid) (color 0 0 0 0))
   )
+  (wire (pts (xy 130.81 101.6) (xy 135.89 101.6))
+    (stroke (width 0) (type solid) (color 0 0 0 0))
+  )
   (wire (pts (xy 196.85 99.06) (xy 199.39 99.06))
     (stroke (width 0) (type solid) (color 0 0 0 0))
   )
+  (wire (pts (xy 130.81 96.52) (xy 135.89 96.52))
+    (stroke (width 0) (type solid) (color 0 0 0 0))
+  )
+  (wire (pts (xy 130.81 106.68) (xy 130.81 114.3))
+    (stroke (width 0) (type solid) (color 0 0 0 0))
+  )
+  (wire (pts (xy 85.09 99.06) (xy 82.55 99.06))
+    (stroke (width 0) (type solid) (color 0 0 0 0))
+  )
   (wire (pts (xy 191.77 90.17) (xy 189.23 90.17))
     (stroke (width 0) (type solid) (color 0 0 0 0))
   )
   (wire (pts (xy 204.47 107.95) (xy 208.28 107.95))
+    (stroke (width 0) (type solid) (color 0 0 0 0))
+  )
+  (wire (pts (xy 82.55 99.06) (xy 82.55 101.6))
+    (stroke (width 0) (type solid) (color 0 0 0 0))
+  )
+  (wire (pts (xy 130.81 99.06) (xy 135.89 99.06))
+    (stroke (width 0) (type solid) (color 0 0 0 0))
+  )
+  (wire (pts (xy 130.81 104.14) (xy 135.89 104.14))
     (stroke (width 0) (type solid) (color 0 0 0 0))
   )
@@
     (effects (font (size 1.27 1.27)) (justify left bottom))
   )
+  (global_label "OLED_SPI_SCK" (shape input) (at 130.81 101.6 180) (fields_autoplaced)
+    (effects (font (size 1.27 1.27)) (justify right))
+    (property "Intersheet References" "${INTERSHEET_REFS}" (id 0) (at 114.9899 101.5206 0)
+      (effects (font (size 1.27 1.27)) (justify right) hide)
+    )
+  )
+  (global_label "OLED_DC" (shape input) (at 130.81 96.52 180) (fields_autoplaced)
+    (effects (font (size 1.27 1.27)) (justify right))
+    (property "Intersheet References" "${INTERSHEET_REFS}" (id 0) (at 120.2514 96.4406 0)
+      (effects (font (size 1.27 1.27)) (justify right) hide)
+    )
+  )
   (global_label "LED-PTT" (shape input) (at 189.23 99.06 180) (fields_autoplaced)
     (effects (font (size 1.27 1.27)) (justify right))
@@
     )
   )
+  (global_label "OLED_SPI_MOSI" (shape input) (at 130.81 104.14 180) (fields_autoplaced)
+    (effects (font (size 1.27 1.27)) (justify right))
+    (property "Intersheet References" "${INTERSHEET_REFS}" (id 0) (at 114.1433 104.0606 0)
+      (effects (font (size 1.27 1.27)) (justify right) hide)
+    )
+  )
   (global_label "LED-SYNC" (shape input) (at 189.23 107.95 180) (fields_autoplaced)
     (effects (font (size 1.27 1.27)) (justify right))
@@
     )
   )
+  (global_label "USART1_RX" (shape input) (at 82.55 93.98 180) (fields_autoplaced)
+    (effects (font (size 1.27 1.27)) (justify right))
+    (property "Intersheet References" "${INTERSHEET_REFS}" (id 0) (at 69.7537 94.0594 0)
+      (effects (font (size 1.27 1.27)) (justify right) hide)
+    )
+  )
+  (global_label "USART1_TX" (shape input) (at 82.55 96.52 180) (fields_autoplaced)
+    (effects (font (size 1.27 1.27)) (justify right))
+    (property "Intersheet References" "${INTERSHEET_REFS}" (id 0) (at 70.0561 96.5994 0)
+      (effects (font (size 1.27 1.27)) (justify right) hide)
+    )
+  )
+  (global_label "OLED_CS" (shape input) (at 130.81 99.06 180) (fields_autoplaced)
+    (effects (font (size 1.27 1.27)) (justify right))
+    (property "Intersheet References" "${INTERSHEET_REFS}" (id 0) (at 120.3118 98.9806 0)
+      (effects (font (size 1.27 1.27)) (justify right) hide)
+    )
+  )
   (global_label "LED-ERROR" (shape input) (at 189.23 116.84 180) (fields_autoplaced)
     (effects (font (size 1.27 1.27)) (justify right))
     (property "Intersheet References" "${INTERSHEET_REFS}" (id 0) (at -72.39 -38.1 0)
       (effects (font (size 1.27 1.27)) hide)
+    )
+  )
+  (global_label "OLED_RST" (shape input) (at 130.81 93.98 180) (fields_autoplaced)
+    (effects (font (size 1.27 1.27)) (justify right))
+    (property "Intersheet References" "${INTERSHEET_REFS}" (id 0) (at 119.3442 93.9006 0)
+      (effects (font (size 1.27 1.27)) (justify right) hide)
     )
   )
@@
     (pin "C")
   )
+  (symbol (lib_id "power:GND") (at 82.55 101.6 0) (unit 1)
+    (in_bom yes) (on_board yes)
+    (property "Reference" "#PWR?" (id 0) (at 82.55 107.95 0)
+      (effects (font (size 1.27 1.27)) hide)
+    )
+    (property "Value" "GND" (id 1) (at 82.677 105.9942 0))
+    (property "Footprint" "" (id 2) (at 82.55 101.6 0)
+      (effects (font (size 1.27 1.27)) hide)
+    )
+    (property "Datasheet" "" (id 3) (at 82.55 101.6 0)
+      (effects (font (size 1.27 1.27)) hide)
+    )
+    (pin "1")
+  )
+  (symbol (lib_id "power:VDD") (at 133.35 91.44 0) (unit 1)
+    (in_bom yes) (on_board yes)
+    (property "Reference" "#PWR?" (id 0) (at 133.35 95.25 0)
+      (effects (font (size 1.27 1.27)) hide)
+    )
+    (property "Value" "VDD" (id 1) (at 133.731 87.0458 0))
+    (property "Footprint" "" (id 2) (at 133.35 91.44 0)
+      (effects (font (size 1.27 1.27)) hide)
+    )
+    (property "Datasheet" "" (id 3) (at 133.35 91.44 0)
+      (effects (font (size 1.27 1.27)) hide)
+    )
+    (pin "1")
+  )
+  (symbol (lib_id "Connector_Generic:Conn_01x07") (at 140.97 101.6 0) (unit 1)
+    (in_bom yes) (on_board yes) (fields_autoplaced)
+    (property "Reference" "J?" (id 0) (at 143.0021 100.6915 0)
+      (effects (font (size 1.27 1.27)) (justify left))
+    )
+    (property "Value" "OLED" (id 1) (at 143.0021 103.4666 0)
+      (effects (font (size 1.27 1.27)) (justify left))
+    )
+    (property "Footprint" "Connector_PinHeader_2.54mm:PinHeader_1x07_P2.54mm_Vertical" (id 2) (at 140.97 101.6 0)
+      (effects (font (size 1.27 1.27)) hide)
+    )
+    (property "Datasheet" "~" (id 3) (at 140.97 101.6 0)
+      (effects (font (size 1.27 1.27)) hide)
+    )
+    (pin "1")
+    (pin "2")
+    (pin "3")
+    (pin "4")
+    (pin "5")
+    (pin "6")
+    (pin "7")
+  )
   (symbol (lib_id "pkl_device:pkl_R_Small") (at 194.31 107.95 270) (unit 1)
     (in_bom yes) (on_board yes)
@@
     (pin "2")
   )
+  (symbol (lib_id "power:GND") (at 130.81 114.3 0) (unit 1)
+    (in_bom yes) (on_board yes)
+    (property "Reference" "#PWR?" (id 0) (at 130.81 120.65 0)
+      (effects (font (size 1.27 1.27)) hide)
+    )
+    (property "Value" "GND" (id 1) (at 130.937 118.6942 0))
+    (property "Footprint" "" (id 2) (at 130.81 114.3 0)
+      (effects (font (size 1.27 1.27)) hide)
+    )
+    (property "Datasheet" "" (id 3) (at 130.81 114.3 0)
+      (effects (font (size 1.27 1.27)) hide)
+    )
+    (pin "1")
+  )
   (symbol (lib_id "power:GND") (at 208.28 119.38 0) (unit 1)
     (in_bom yes) (on_board yes)
@@
     (pin "1")
   )
+  (symbol (lib_id "Connector_Generic:Conn_01x03") (at 90.17 96.52 0) (unit 1)
+    (in_bom yes) (on_board yes) (fields_autoplaced)
+    (property "Reference" "J?" (id 0) (at 92.2021 95.6115 0)
+      (effects (font (size 1.27 1.27)) (justify left))
+    )
+    (property "Value" "UART" (id 1) (at 92.2021 98.3866 0)
+      (effects (font (size 1.27 1.27)) (justify left))
+    )
+    (property "Footprint" "Connector_PinHeader_2.54mm:PinHeader_1x03_P2.54mm_Vertical" (id 2) (at 90.17 96.52 0)
+      (effects (font (size 1.27 1.27)) hide)
+    )
+    (property "Datasheet" "~" (id 3) (at 90.17 96.52 0)
+      (effects (font (size 1.27 1.27)) hide)
+    )
+    (pin "1")
+    (pin "2")
+    (pin "3")
+  )
 )

Commit message: RF part update
Parts:
- R25, R26, R27, R28: renamed from R?; footprint pkl_dipol:R_0603 -> Resistor_SMD:R_0402_1005Metric
- gave numbers to parts that had none: 6
Changed lines of the file:
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@@
   (symbol (lib_id "pkl_device:pkl_R_Small") (at 194.31 116.84 270) (unit 1)
     (in_bom yes) (on_board yes)
-    (property "Reference" "R?" (id 0) (at 194.31 111.76 90))
+    (property "Reference" "R28" (id 0) (at 194.31 111.76 90))
     (property "Value" "680R" (id 1) (at 194.31 114.173 90))
-    (property "Footprint" "pkl_dipol:R_0603" (id 2) (at 194.31 116.84 0)
+    (property "Footprint" "Resistor_SMD:R_0402_1005Metric" (id 2) (at 194.31 116.84 0)
       (effects (font (size 1.524 1.524)) hide)
     )
@@
   (symbol (lib_id "pkl_device:pkl_Led_Small") (at 201.93 116.84 0) (unit 1)
     (in_bom yes) (on_board yes)
-    (property "Reference" "D?" (id 0) (at 201.93 110.871 0))
+    (property "Reference" "D8" (id 0) (at 201.93 110.871 0))
     (property "Value" "Error" (id 1) (at 201.93 113.1824 0))
     (property "Footprint" "pkl_dipol:D_0603" (id 2) (at 201.93 116.84 90)
@@
   (symbol (lib_id "pkl_device:pkl_Led_Small") (at 201.93 99.06 0) (unit 1)
     (in_bom yes) (on_board yes)
-    (property "Reference" "D?" (id 0) (at 201.93 93.091 0))
+    (property "Reference" "D6" (id 0) (at 201.93 93.091 0))
     (property "Value" "PTT" (id 1) (at 201.93 95.4024 0))
     (property "Footprint" "pkl_dipol:D_0603" (id 2) (at 201.93 99.06 90)
@@
   (symbol (lib_id "pkl_device:pkl_Led_Small") (at 201.93 107.95 0) (unit 1)
     (in_bom yes) (on_board yes)
-    (property "Reference" "D?" (id 0) (at 201.93 101.981 0))
+    (property "Reference" "D7" (id 0) (at 201.93 101.981 0))
     (property "Value" "Sync" (id 1) (at 201.93 104.2924 0))
     (property "Footprint" "pkl_dipol:D_0603" (id 2) (at 201.93 107.95 90)
@@
   (symbol (lib_id "pkl_device:pkl_Led_Small") (at 201.93 90.17 0) (unit 1)
     (in_bom yes) (on_board yes)
-    (property "Reference" "D?" (id 0) (at 201.93 84.201 0))
+    (property "Reference" "D5" (id 0) (at 201.93 84.201 0))
     (property "Value" "Power" (id 1) (at 201.93 86.5124 0))
     (property "Footprint" "pkl_dipol:D_0603" (id 2) (at 201.93 90.17 90)
@@
   (symbol (lib_id "power:GND") (at 82.55 101.6 0) (unit 1)
     (in_bom yes) (on_board yes)
-    (property "Reference" "#PWR?" (id 0) (at 82.55 107.95 0)
+    (property "Reference" "#PWR0197" (id 0) (at 82.55 107.95 0)
       (effects (font (size 1.27 1.27)) hide)
     )
@@
   (symbol (lib_id "power:VDD") (at 133.35 91.44 0) (unit 1)
     (in_bom yes) (on_board yes)
-    (property "Reference" "#PWR?" (id 0) (at 133.35 95.25 0)
+    (property "Reference" "#PWR0198" (id 0) (at 133.35 95.25 0)
       (effects (font (size 1.27 1.27)) hide)
     )
@@
   (symbol (lib_id "Connector_Generic:Conn_01x07") (at 140.97 101.6 0) (unit 1)
     (in_bom yes) (on_board yes) (fields_autoplaced)
-    (property "Reference" "J?" (id 0) (at 143.0021 100.6915 0)
+    (property "Reference" "J7" (id 0) (at 143.0021 100.6915 0)
       (effects (font (size 1.27 1.27)) (justify left))
     )
@@
   (symbol (lib_id "pkl_device:pkl_R_Small") (at 194.31 107.95 270) (unit 1)
     (in_bom yes) (on_board yes)
-    (property "Reference" "R?" (id 0) (at 194.31 102.87 90))
+    (property "Reference" "R27" (id 0) (at 194.31 102.87 90))
     (property "Value" "680R" (id 1) (at 194.31 105.283 90))
-    (property "Footprint" "pkl_dipol:R_0603" (id 2) (at 194.31 107.95 0)
+    (property "Footprint" "Resistor_SMD:R_0402_1005Metric" (id 2) (at 194.31 107.95 0)
       (effects (font (size 1.524 1.524)) hide)
     )
@@
   (symbol (lib_id "pkl_device:pkl_R_Small") (at 194.31 90.17 270) (unit 1)
     (in_bom yes) (on_board yes)
-    (property "Reference" "R?" (id 0) (at 194.31 85.09 90))
+    (property "Reference" "R25" (id 0) (at 194.31 85.09 90))
     (property "Value" "680R" (id 1) (at 194.31 87.503 90))
-    (property "Footprint" "pkl_dipol:R_0603" (id 2) (at 194.31 90.17 0)
+    (property "Footprint" "Resistor_SMD:R_0402_1005Metric" (id 2) (at 194.31 90.17 0)
       (effects (font (size 1.524 1.524)) hide)
     )
@@
   (symbol (lib_id "pkl_device:pkl_R_Small") (at 194.31 99.06 270) (unit 1)
     (in_bom yes) (on_board yes)
-    (property "Reference" "R?" (id 0) (at 194.31 93.98 90))
+    (property "Reference" "R26" (id 0) (at 194.31 93.98 90))
     (property "Value" "680R" (id 1) (at 194.31 96.393 90))
-    (property "Footprint" "pkl_dipol:R_0603" (id 2) (at 194.31 99.06 0)
+    (property "Footprint" "Resistor_SMD:R_0402_1005Metric" (id 2) (at 194.31 99.06 0)
       (effects (font (size 1.524 1.524)) hide)
     )
@@
   (symbol (lib_id "power:GND") (at 130.81 114.3 0) (unit 1)
     (in_bom yes) (on_board yes)
-    (property "Reference" "#PWR?" (id 0) (at 130.81 120.65 0)
+    (property "Reference" "#PWR0196" (id 0) (at 130.81 120.65 0)
       (effects (font (size 1.27 1.27)) hide)
     )
@@
   (symbol (lib_id "power:GND") (at 208.28 119.38 0) (unit 1)
     (in_bom yes) (on_board yes)
-    (property "Reference" "#PWR?" (id 0) (at 208.28 125.73 0)
+    (property "Reference" "#PWR0195" (id 0) (at 208.28 125.73 0)
       (effects (font (size 1.27 1.27)) hide)
     )
@@
   (symbol (lib_id "Connector_Generic:Conn_01x03") (at 90.17 96.52 0) (unit 1)
     (in_bom yes) (on_board yes) (fields_autoplaced)
-    (property "Reference" "J?" (id 0) (at 92.2021 95.6115 0)
+    (property "Reference" "J6" (id 0) (at 92.2021 95.6115 0)
       (effects (font (size 1.27 1.27)) (justify left))
     )
