File: mcu.kicad_sch (KiCad schematic)
At the start: 18 parts

Commit message: Add files via upload
Parts:
- added C? (x2): 12p, pkl_dipol:C_0603, symbol pkl_device:pkl_C_Small
- added J?: STLink, Connector_PinHeader_2.54mm:PinHeader_1x04_P2.54mm_Vertical, symbol Connector_Generic:Conn_01x04
- added R? (x2): 22, pkl_dipol:R_0603, symbol pkl_device:pkl_R_Small
- added Y?: 32 kHz, Crystal:Crystal_SMD_MicroCrystal_CC8V-T1A-2Pin_2.0x1.2mm, symbol Device:Crystal_Small
Connections:
- net GND: now also C?.2, C?.2, J?.4 (Pin_4)
- net NRST: now also J?.3 (Pin_3)
- new net: J?.1 (Pin_1), R?.2
- new net: J?.2 (Pin_2), R?.2
- new net RTC_X1: C?.1, Y?.1
- new net RTC_X2: C?.1, Y?.2
- new net SWCLK: R?.1
- new net SWDIO: R?.1
Other:
- note added: "Add some caps here"
- moved on the sheet: J?

Commit message: RF part update
Parts:
- C2, C3, C4, C5: renamed from C?; footprint pkl_dipol:C_0603 -> Capacitor_SMD:C_0402_1005Metric
- J2: renamed from J?; footprint (none) -> Connector_Card:microSD_HC_Hirose_DM3AT-SF-PEJM5
- R3, R4, R5, R6, R7, R8: renamed from R?; footprint pkl_dipol:R_0603 -> Resistor_SMD:R_0402_1005Metric
- gave numbers to parts that had none: 13
