File: power.kicad_sch (KiCad schematic)
At the start: 20 parts

Commit message: Add files via upload
Parts:
- added C? (x3): 100n, pkl_dipol:C_0603, symbol pkl_device:pkl_C_Small
- added C?: 10u, Capacitor_Tantalum_SMD:CP_EIA-3216-18_Kemet-A, symbol pkl_device:pkl_CP_Small
- added C?: 1u, pkl_dipol:C_0603, symbol pkl_device:pkl_C_Small
- added C?: 22u, Capacitor_SMD:C_1210_3225Metric, symbol pkl_device:pkl_C_Small
- added C?: 10u, Capacitor_SMD:C_1210_3225Metric, symbol pkl_device:pkl_C_Small
- added C?: 10n, pkl_dipol:C_0603, symbol pkl_device:pkl_C_Small
- added D?: DFLT18A-7, Diode_SMD:D_SOD-128, symbol Device:D_Zener_Small
- added F?: Polyfuse, symbol Device:Polyfuse
- added FB?: FB0805, pkl_dipol:L_0805, symbol Device:Ferrite_Bead_Small
- added L?: 10u, Inductor_SMD:L_Vishay_IHLP-2525, symbol pkl_device:pkl_L_Small
- added R?: 100k, pkl_dipol:R_0603, symbol pkl_device:pkl_R_Small
- added R?: 126k, pkl_dipol:R_0603, symbol pkl_device:pkl_R_Small
- added R?: 24k, pkl_dipol:R_0603, symbol pkl_device:pkl_R_Small
- added RV?: 50k, M17-SmartMic:PTR901, symbol M17-SmartMic:R_Potentiometer_Switch
- added U?: TPS73233, Package_TO_SOT_SMD:SOT-23-5, symbol Regulator_Linear:TPS73133DBV
- added U?: TP6841S6, Package_TO_SOT_SMD:SOT-23-6, symbol Module17:TP6841S6
Connections:
- net GND: now also C?.1, C?.2, C?.2, C?.2, C?.2, C?.2, C?.2, D?.2 (A), R?.1, U?.2 (GND), U?.2 (GND)
- net VBAT: now also RV?.SW1 (SW)
- net VDD: now also C?.1, C?.1, U?.5 (OUT)
- new net: C?.1, FB?.1, R?.1, U?.5 (VIN)
- new net: R?.2, U?.4 (EN)
- new net: C?.2, D?.1 (K), F?.2, FB?.2
- new net: C?.2, L?.2, U?.6 (SW)
- new net: R?.1, R?.2, U?.3 (FB)
- new net: C?.1, U?.1 (BST)
- new net: F?.1, RV?.SW2 (SW)
- new net +5V: C?.1, C?.1, C?.1, L?.1, R?.2, U?.1 (IN), U?.3 (EN)
Other:
- moved on the sheet: BT?, C?, D?, FB?, H?, R?

Commit message: RF part update
Parts:
- C29, C30, C31, C32, C33, C34, C35, C36, C38, C39, C40, C43, C45, C46: renamed from C?; footprint pkl_dipol:C_0603 -> Capacitor_SMD:C_0402_1005Metric
- C37: renamed from C?; footprint Capacitor_SMD:C_1210_3225Metric -> Capacitor_SMD:C_0603_1608Metric
- F1: renamed from F?; footprint (none) -> Fuse:Fuse_0805_2012Metric
- R20, R21, R22, R23, R24: renamed from R?; footprint pkl_dipol:R_0603 -> Resistor_SMD:R_0402_1005Metric
- gave numbers to parts that had none: 17
