File: rf.kicad_sch (KiCad schematic)
At the start: 10 parts

Commit message: RF part update
Parts:
- added C47, C48, C53: 5.1p, Capacitor_SMD:C_0402_1005Metric, symbol pkl_device:pkl_C_Small
- added C49: 39p, Capacitor_SMD:C_0402_1005Metric, symbol pkl_device:pkl_C_Small
- added C50: 56p, Capacitor_SMD:C_0402_1005Metric, symbol pkl_device:pkl_C_Small
- added C51: 2.2p, Capacitor_SMD:C_0402_1005Metric, symbol pkl_device:pkl_C_Small
- added C52: 10n, Capacitor_SMD:C_0402_1005Metric, symbol pkl_device:pkl_C_Small
- added C54: 6.2p, Capacitor_SMD:C_0402_1005Metric, symbol pkl_device:pkl_C_Small
- added C55: 100p, Capacitor_SMD:C_0402_1005Metric, symbol pkl_device:pkl_C_Small
- added J8: Conn_Coaxial, symbol Connector:Conn_Coaxial
- added L2, L4: 27n, Inductor_SMD:L_0402_1005Metric, symbol Device:L_Small
- added L3, L6: 56n, Inductor_SMD:L_0402_1005Metric, symbol Device:L_Small
- added L5, L7: 15n, Inductor_SMD:L_0402_1005Metric, symbol Device:L_Small
- added L8: 43n, Inductor_SMD:L_0402_1005Metric, symbol Device:L_Small
- added L9: 22n, Inductor_SMD:L_0402_1005Metric, symbol Device:L_Small
- added R29: 18, Resistor_SMD:R_0402_1005Metric, symbol pkl_device:pkl_R_Small
- C10, C11, C12, C13, C14, C8, C9: renamed from C?; footprint pkl_dipol:C_0603 -> Capacitor_SMD:C_0402_1005Metric
- R9: renamed from R?; footprint pkl_dipol:R_0603 -> Resistor_SMD:R_0402_1005Metric
- gave numbers to parts that had none: 2
Connections:
- net GND: now also C48.2, C52.2, C54.2, C55.2, J8.2 (Ext), L2.2
- net VDD: now also C50.1, C52.1, C55.1, R29.1
- net PA: now reaches U4.17 (PA)
- net PA: now also C49.2, L6.2
- net TRX_SW: now reaches U4.18 (TRX_SW)
- net TRX_SW: now also C53.2, L5.1
- net LNA_P: now reaches U4.19 (LNA_P)
- net LNA_P: now also C47.1, L2.1, L3.1
- net LNA_N: now reaches U4.20 (LNA_N)
- net LNA_N: now also C48.1, L3.2, L4.1
- new net: C54.1, L8.2, L9.1
- new net: C51.1, C53.1, L7.2, L8.1
- new net: C50.2, L6.1, R29.2
- new net: C49.1, C51.2, L7.1
- new net: C47.2, L4.2, L5.2
- new net: J8.1 (In), L9.2
Other:
- moved on the sheet: C10, C11, C12, C13, C14, C8, C9, R9, U4, Y3
