File: Hardware/KiCad/Mini17.kicad_pcb (KiCad board)
At the start: 2 copper layers, 180 parts, among them IC1 LM4861M, J1 USB_C, J2 STLink, J3 Micro_SD_Card_Det, J4 Kenwood-3.5, J5 Kenwood-2.5, J6 UART, J7 OLED, J8 Conn_Coaxial, SW1 PTT, SW10 SW_Push_45deg, SW11 SW_Push_45deg, SW12 SW_Push_45deg, SW13 SW_Push_45deg, SW14 SW_Push_45deg, SW15 SW_Push_45deg, SW16 SW_Push_45deg, SW17 SW_Push_45deg, SW2 SW_Push_45deg, SW3 SW_Push_45deg, SW4 SW_Push_45deg, SW5 SW_Push_45deg, SW6 SW_Push_45deg, SW7 SW_Push_45deg, SW8 SW_Push_45deg, SW9 SW_Push_45deg, U1 USBLC6-2, U3 STM32F427ZGTx, U4 CC1200, U5 MAX9814, U6 TP6841S6, U7 TPS73233, Y1 8 MHz, Y3 40 MHz

Commit message: add fpc display board connector, move components around, rough size of board
Parts:
- removed the D6 at (75.3, 70.9)
- added C1: 10nF, Capacitor_SMD:C_0402_1005Metric, F.Cu at (77.1, 304.7)
- added C12: 10nF, Capacitor_SMD:C_0402_1005Metric, F.Cu at (71.3, 308.7)
- added C13: 100nF, Capacitor_SMD:C_0402_1005Metric, F.Cu at (74.2, 304.7)
- added C14: 100n, Capacitor_SMD:C_0402_1005Metric, F.Cu at (74.2, 306.7)
- added C29: 100n, Capacitor_SMD:C_0402_1005Metric, F.Cu at (71.3, 306.7)
- added C8: 10nF, Capacitor_SMD:C_0402_1005Metric, F.Cu at (68.4, 308.7)
- added FB3: BLM18AG601SN1D, digikey-footprints:0603, F.Cu at (92.8, 307.0)
- added J9: Front Panel Connector, SamacSys_Parts3:FH19SC24S05SH09, F.Cu at (120.1, 120.7)
- added R29: 10k, Resistor_SMD:R_0402_1005Metric, F.Cu at (62.6, 306.7)
- added R36: 10k, Resistor_SMD:R_0402_1005Metric, F.Cu at (68.4, 304.7)
- added R37: 10k, Resistor_SMD:R_0402_1005Metric, F.Cu at (65.5, 308.7)
- added R38: 10k, Resistor_SMD:R_0402_1005Metric, F.Cu at (83.8, 296.1)
- added R39: 47k, Resistor_SMD:R_0402_1005Metric, F.Cu at (83.8, 298.0)
- added R40: 10k, Resistor_SMD:R_0402_1005Metric, F.Cu at (68.4, 306.7)
- added R41: 10k, Resistor_SMD:R_0402_1005Metric, F.Cu at (65.5, 306.7)
- added R42: 10k, Resistor_SMD:R_0402_1005Metric, F.Cu at (62.6, 304.7)
- added R43: 10k, Resistor_SMD:R_0402_1005Metric, F.Cu at (62.6, 308.7)
- added R8: 10k, Resistor_SMD:R_0402_1005Metric, F.Cu at (71.4, 304.7)
- added R9: 10k, Resistor_SMD:R_0402_1005Metric, F.Cu at (65.5, 304.7)
- added SW19: F1, Button_Switch_THT:SW_Tactile_SPST_Angled_PTS645Vx31-2LFS, F.Cu at (67.6, 136.9)
- added SW20: F2, Button_Switch_THT:SW_Tactile_SPST_Angled_PTS645Vx31-2LFS, F.Cu at (55.9, 136.9)
- added TP10: TP_5V, TestPoint:TestPoint_Pad_D1.0mm, F.Cu at (68.8, 314.7)
- added TP11: TP_3V3, TestPoint:TestPoint_Pad_D1.0mm, F.Cu at (65.7, 314.7)
- added TP12: TP_BAT_ADC, TestPoint:TestPoint_Pad_D1.0mm, F.Cu at (62.7, 314.7)
- added TP13: TP_SPK_P, TestPoint:TestPoint_Pad_D1.0mm, F.Cu at (96.1, 307.3)
- added TP5: TP_B, TestPoint:TestPoint_Pad_D1.0mm, F.Cu at (75.8, 314.7)
- added TP6: TP_A, TestPoint:TestPoint_Pad_D1.0mm, F.Cu at (78.9, 314.7)
- added TP7: TP_CC0, TestPoint:TestPoint_Pad_D1.0mm, F.Cu at (95.6, 296.6)
- added TP8: TP_CC2, TestPoint:TestPoint_Pad_D1.0mm, F.Cu at (92.5, 299.6)
- added TP9: TP_CC3, TestPoint:TestPoint_Pad_D1.0mm, F.Cu at (92.5, 296.6)
- C10: value 220n -> 220p
- C27: value 470u -> 100u/6.3V; footprint Capacitor_SMD:CP_Elec_6.3x7.7 -> Capacitor_SMD:C_1206_3216Metric
- J1: footprint Connector_USB:USB_C_Receptacle_HRO_TYPE-C-31-M-12 -> Connector_USB:USB_C_Receptacle_GCT_USB4085; moved to B.Cu
- J3, J4, J5, U1: moved to B.Cu
- TP4: value TP_SPK -> TP_SPK_N
- moved J8 226.1 mm to (40.6, 107.9), turned to 90 degrees
- moved L174 214.1 mm to (46.6, 107.9), turned to 180 degrees
- moved C175 211.1 mm to (48.1, 107.4), turned to 90 degrees
- moved L173 208.1 mm to (49.6, 107.9), turned to 180 degrees
- moved L192 205.6 mm to (50.7, 111.7), turned to 180 degrees
- moved C181 205.0 mm to (51.1, 108.3), turned to -90 degrees
- moved L193 204.9 mm to (51.1, 110.2), turned to -90 degrees
- moved J2 204.6 mm to (32.2, -97.7)
- moved L201 203.5 mm to (51.8, 112.8), turned to 180 degrees
- moved C201 203.5 mm to (51.8, 113.8), turned to 180 degrees
- moved C191 202.7 mm to (52.2, 111.3), turned to 90 degrees
- moved C176 202.1 mm to (52.6, 107.9), turned to 0 degrees
- moved L191 200.5 mm to (53.3, 112.3), turned to -90 degrees
- moved L172 199.0 mm to (54.1, 108.3), turned to -90 degrees
- moved C174 196.1 mm to (55.6, 107.9), turned to 0 degrees
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Connections:
- net INT_SPEAKER renamed INT_SPK
- net Net-(C26-Pad1) renamed SPK_P
- C27 pad 2: EXT_SPEAKER -> SPK_N
- D5 pad 1: (no net) -> GND
- D5 pad 2: (no net) -> Net-(D5-Pad2)
- J2 pad 4: GND -> unconnected-(J2-Pad4)
- LS1 pad 2: GND -> SPK_N
- R15 pad 1: ~{PTT_IN} -> PTT_IN
- R25 pad 1: Net-(D5-PadA) -> Net-(D5-Pad2)
- R5 pad 2: USB_DN -> USB_DM
- TP4 pad 1: EXT_SPEAKER -> SPK_N
- U3 pad 114: unconnected-(U3-Pad114) -> SD_DET
- U3 pad 138: ~{BOOT0} -> BOOT0
- U3 pad 141: unconnected-(U3-Pad141) -> Net-(TP6-Pad1)
- U3 pad 142: unconnected-(U3-Pad142) -> Net-(TP5-Pad1)
- U3 pad 22: unconnected-(U3-Pad22) -> BOOT0
- U3 pad 26: unconnected-(U3-Pad26) -> BTN_F1
- U3 pad 27: unconnected-(U3-Pad27) -> PTT_IN
- U3 pad 41: LED-PTT -> LED_PTT
- U3 pad 5: LED-SYNC -> LED_SYNC
- U3 pad 81: LED-ERROR -> LED_ERR
- U3 pad 93: unconnected-(U3-Pad93) -> ENC_BTN
- U3 pad 96: unconnected-(U3-Pad96) -> ENC_B
- U3 pad 97: SD_DET -> ENC_A
Routing:
- net GND: track 27.3 -> 16.8 mm, vias 0 -> 2
- net CC_X2: track 0.00 -> 7.90 mm
- net CC_X1: track 0.00 -> 6.52 mm
- net Net-(C291-Pad1): track 0.00 -> 4.32 mm
- net Net-(C5-Pad2): track 0.00 -> 3.20 mm
- net Net-(C4-Pad2): track 0.00 -> 2.74 mm
- net XTAL_1: track 7.34 -> 9.71 mm
- net XTAL_2: track 5.50 -> 7.29 mm
- net Net-(C231-Pad2): track 3.19 -> 2.44 mm
- net Net-(C231-Pad1): track 3.01 -> 2.31 mm
Other:
- board outline added: 99.6 x 43.7 mm
- copper layers 2 -> 4

Commit message: many edits throughout, added board edges for main & HMI combined, added rough layouts for some components on both
Parts:
- removed H1, H2, H3, H4: M2, MountingHole:MountingHole_2.2mm_M2_DIN965_Pad
- removed J4: Kenwood-3.5, M17-SmartMic:PJ-3136-B
- removed J5: Kenwood-2.5, M17-SmartMic:PJ-211A
- removed J7: OLED, Connector_PinHeader_2.54mm:PinHeader_1x07_P2.54mm_Vertical
- removed J9: Front Panel Connector, SamacSys_Parts3:FH19SC24S05SH09
- removed SW10, SW11, SW12, SW13, SW14, SW15, SW16, SW17, SW2, SW3, SW4, SW5, SW6, SW7, SW8, SW9: SW_Push_45deg, Button_Switch_SMD:SW_Push_1P1T_NO_CK_KMR2
- removed SW19: F1, Button_Switch_THT:SW_Tactile_SPST_Angled_PTS645Vx31-2LFS
- removed SW20: F2, Button_Switch_THT:SW_Tactile_SPST_Angled_PTS645Vx31-2LFS
- added ? (x2): , , F.Cu at (149.9, 71.1)
- added ?: , , F.Cu at (145.6, 37.6)
- added ? (x2): , , F.Cu at (149.9, 119.9)
- added ? (x2): , , F.Cu at (149.9, 63.0)
- added ?: , , F.Cu at (149.9, 115.8)
- added ? (x2): , , F.Cu at (149.9, 95.5)
- added ? (x2): , , F.Cu at (149.9, 87.4)
- added ? (x2): , , F.Cu at (149.9, 103.6)
- added ? (x2): , , F.Cu at (149.9, 111.8)
- added ? (x2): , , F.Cu at (149.9, 54.9)
- added ? (x2): , , F.Cu at (149.9, 38.6)
- added ? (x2): , , F.Cu at (149.9, 79.2)
- added ? (x2): , , F.Cu at (149.9, 50.8)
- added ? (x2): , , F.Cu at (149.9, 58.9)
- added ?: , , F.Cu at (145.6, 138.9)
- added ? (x2): , , F.Cu at (149.9, 107.7)
- added ?: , , F.Cu at (105.0, 138.9)
- added ?: , , F.Cu at (105.2, 37.6)
- added ?: , , F.Cu at (149.9, 42.7)
- added ?: , , F.Cu at (194.1, 37.6)
- added ? (x2): , , F.Cu at (149.9, 46.7)
- added ? (x2): , , F.Cu at (149.9, 99.6)
- added ?: , , F.Cu at (149.9, 136.1)
- added ?: , , F.Cu at (149.9, 132.1)
- added ? (x2): , , F.Cu at (149.9, 124.0)
- added ?: , , F.Cu at (149.9, 91.4)
- added ?: , , F.Cu at (153.5, 138.9)
- added ? (x2): , , F.Cu at (149.9, 75.2)
- added ? (x2): , , F.Cu at (149.9, 83.3)
- added ?: , , F.Cu at (149.9, 128.0)
- added ?: , , F.Cu at (153.7, 37.6)
- added ?: , , F.Cu at (149.9, 67.1)
- added ?: , , F.Cu at (194.1, 138.9)
- added C1001: 10n, Capacitor_SMD:C_0603_1608Metric, F.Cu at (330.5, 421.4)
- added C1002: 100n, Capacitor_SMD:C_0603_1608Metric, F.Cu at (338.6, 412.9)
- added C1003: 100n, Capacitor_SMD:C_0603_1608Metric, F.Cu at (333.1, 416.4)
- added C1004: 100n, Capacitor_SMD:C_0603_1608Metric, F.Cu at (322.4, 420.3)
- added C1005: 100n, Capacitor_SMD:C_0603_1608Metric, F.Cu at (334.6, 413.5)
- added C1006: 1u, Capacitor_SMD:C_0603_1608Metric, F.Cu at (320.3, 430.0)
- added C1007: 1u, Capacitor_SMD:C_0603_1608Metric, F.Cu at (344.0, 407.1)
- added C1008: 1u, Capacitor_SMD:C_0603_1608Metric, F.Cu at (334.6, 411.0)
- added C1009: 1u, Capacitor_SMD:C_0603_1608Metric, F.Cu at (330.5, 418.9)
- added C1010: 1u, Capacitor_SMD:C_0603_1608Metric, F.Cu at (313.7, 432.9)
- added C1011: 100n, Capacitor_SMD:C_0603_1608Metric, F.Cu at (326.4, 420.3)
- added C1012: 100n, Capacitor_SMD:C_0603_1608Metric, F.Cu at (329.1, 416.4)
- added C2001: 100nF, Capacitor_SMD:C_0402_1005Metric, F.Cu at (288.7, 442.6)
- added C8001: 100n, Capacitor_SMD:C_0402_1005Metric, F.Cu at (333.9, 418.6)
- added C8002: 100n, Capacitor_SMD:C_0402_1005Metric, F.Cu at (342.0, 409.3)
- added D1001: LED, Diode_SMD:D_0603_1608Metric, F.Cu at (286.4, 436.0)
- added D1002: LED, Diode_SMD:D_0603_1608Metric, F.Cu at (290.5, 436.0)
- added FB1001: Ferrite_Bead, Inductor_SMD:L_0603_1608Metric, F.Cu at (339.9, 407.1)
- added FB1002: Ferrite_Bead, Inductor_SMD:L_0603_1608Metric, F.Cu at (345.9, 404.2)
- added H1001: M2, MountingHole:MountingHole_2.2mm_M2_ISO14580_Pad, F.Cu at (328.4, 437.4)
- added H1002: M2, MountingHole:MountingHole_2.2mm_M2_ISO14580_Pad, F.Cu at (345.2, 438.4)
- added H1003: M2, MountingHole:MountingHole_2.2mm_M2_ISO14580_Pad, F.Cu at (336.0, 437.4)
- added H1004: M2, MountingHole:MountingHole_2.2mm_M2_ISO14580_Pad, F.Cu at (355.3, 438.4)
- added J10: MIC_EXT, TR-9:MIC_EXT, F.Cu at (195.1, 80.5)
- added J1001: Boot0, Connector_PinHeader_2.54mm:PinHeader_1x02_P2.54mm_Vertical, B.Cu at (155.4, 77.5)
- added J1002: SWD, Connector_PinHeader_1.27mm:PinHeader_1x04_P1.27mm_Vertical, B.Cu at (155.7, 89.5)
- added J1003: FH12-22S-0.5SH, Connector_FFC-FPC:Hirose_FH12-22S-0.5SH_1x22-1MP_P0.50mm_Horizontal, B.Cu at (172.5, 76.0)
- added J1004: MainBoard, Connector_FFC-FPC:Hirose_FH12-10S-0.5SH_1x10-1MP_P0.50mm_Horizontal, B.Cu at (160.0, 113.0)
- added J12: SPK_EXT, TR-9:SPK_EXT, F.Cu at (195.3, 72.9)
- added J6001: HMI, Connector_FFC-FPC:Hirose_FH12-10S-0.5SH_1x10-1MP_P0.50mm_Horizontal, F.Cu at (107.5, 113.0)
- added R1001: 10k, Resistor_SMD:R_0603_1608Metric, F.Cu at (317.7, 432.9)
- added R1002: 47R, Resistor_SMD:R_0603_1608Metric, F.Cu at (345.9, 401.7)
- added R1003: 47k, Resistor_SMD:R_0603_1608Metric, F.Cu at (325.7, 422.8)
- added R1004: 47k, Resistor_SMD:R_0603_1608Metric, F.Cu at (325.7, 425.3)
- added R1005: 47k, Resistor_SMD:R_0603_1608Metric, F.Cu at (309.7, 437.1)
- added R1006: 47k, Resistor_SMD:R_0603_1608Metric, F.Cu at (313.8, 435.4)
- added R1007: 47k, Resistor_SMD:R_0603_1608Metric, F.Cu at (305.7, 437.1)
- added R1008: 47k, Resistor_SMD:R_0603_1608Metric, F.Cu at (349.9, 401.7)
- added R1009: 47k, Resistor_SMD:R_0603_1608Metric, F.Cu at (338.6, 410.4)
- added R1010: 47k, Resistor_SMD:R_0603_1608Metric, F.Cu at (320.3, 427.5)
- added R2001: 47k, Resistor_SMD:R_0402_1005Metric, F.Cu at (285.8, 442.6)
- added R6001: 10k, Resistor_SMD:R_0603_1608Metric, F.Cu at (369.3, 401.7)
- added R8001: 10k, Resistor_SMD:R_0402_1005Metric, F.Cu at (317.2, 435.1)
- added R8002: 10k, Resistor_SMD:R_0402_1005Metric, F.Cu at (336.6, 415.8)
- added R8003: 10k, Resistor_SMD:R_0402_1005Metric, F.Cu at (300.9, 410.4)
- added R8004: 10k, Resistor_SMD:R_0402_1005Metric, F.Cu at (298.0, 410.4)
- added SW1002: SW_Push, Button_Switch_SMD:SW_Push_1P1T_NO_CK_KMR2, F.Cu at (161.8, 97.0)
- added SW1003: SW_Push, Button_Switch_SMD:SW_Push_1P1T_NO_CK_KMR2, F.Cu at (161.8, 103.9)
- added SW1004: SW_Push, Button_Switch_SMD:SW_Push_1P1T_NO_CK_KMR2, F.Cu at (161.8, 111.0)
- added SW1005: SW_Push, Button_Switch_SMD:SW_Push_1P1T_NO_CK_KMR2, F.Cu at (161.8, 118.1)
- added SW1006: SW_Push, Button_Switch_SMD:SW_Push_1P1T_NO_CK_KMR2, F.Cu at (161.8, 125.0)
- added SW1007: SW_Push, Button_Switch_SMD:SW_Push_1P1T_NO_CK_KMR2, F.Cu at (161.8, 132.1)
- added SW1008: SW_Push, Button_Switch_SMD:SW_Push_1P1T_NO_CK_KMR2, F.Cu at (172.7, 97.0)
- added SW1009: SW_Push, Button_Switch_SMD:SW_Push_1P1T_NO_CK_KMR2, F.Cu at (172.7, 103.9)
- added SW1010: SW_Push, Button_Switch_SMD:SW_Push_1P1T_NO_CK_KMR2, F.Cu at (172.7, 111.0)
- added SW1011: SW_Push, Button_Switch_SMD:SW_Push_1P1T_NO_CK_KMR2, F.Cu at (172.7, 117.9)
- added SW1012: SW_Push, Button_Switch_SMD:SW_Push_1P1T_NO_CK_KMR2, F.Cu at (172.7, 125.0)
- added SW1013: SW_Push, Button_Switch_SMD:SW_Push_1P1T_NO_CK_KMR2, F.Cu at (172.7, 131.8)
- added SW1015: SW_Push, Button_Switch_SMD:SW_Push_1P1T_NO_CK_KMR2, F.Cu at (183.9, 97.0)
- added SW1016: SW_Push, Button_Switch_SMD:SW_Push_1P1T_NO_CK_KMR2, F.Cu at (183.9, 103.9)
- added SW1017: SW_Push, Button_Switch_SMD:SW_Push_1P1T_NO_CK_KMR2, F.Cu at (183.9, 111.0)
- added SW1018: SW_Push, Button_Switch_SMD:SW_Push_1P1T_NO_CK_KMR2, F.Cu at (183.9, 117.9)
- added SW1019: SW_Push, Button_Switch_SMD:SW_Push_1P1T_NO_CK_KMR2, F.Cu at (183.9, 125.0)
- added SW1020: SW_Push, Button_Switch_SMD:SW_Push_1P1T_NO_CK_KMR2, F.Cu at (184.2, 131.8)
- added SW8001: F1, Button_Switch_THT:SW_Tactile_SPST_Angled_PTS645Vx31-2LFS, F.Cu at (194.9, 52.8)
- added SW8002: F2, Button_Switch_THT:SW_Tactile_SPST_Angled_PTS645Vx31-2LFS, F.Cu at (194.9, 42.9)
- added TP1001: TestPoint, TestPoint:TestPoint_Pad_2.0x2.0mm, F.Cu at (321.7, 423.6)
- added TP1002: TestPoint, TestPoint:TestPoint_Pad_2.0x2.0mm, F.Cu at (335.9, 407.1)
- added TP1003: TestPoint, TestPoint:TestPoint_Pad_2.0x2.0mm, F.Cu at (301.7, 436.5)
- added U1001: STM32F030K6Tx, Package_QFP:LQFP-32_7x7mm_P0.8mm, B.Cu at (172.0, 90.9)
- added X1001: ASV-4.000MHZ-EJ-T, Oscillator:Oscillator_SMD_Abracon_ASV-4Pin_7.0x5.1mm, B.Cu at (184.2, 89.7)
- C1: value 220n -> 10nF
- C8: value 4.7u -> 10nF
- J1, U1: moved to F.Cu
- J3: footprint Connector_Card:microSD_HC_Hirose_DM3AT-SF-PEJM5 -> Connector_USB:USB_Mini-B_Wuerth_65100516121_Horizontal; moved to F.Cu
- R8: value 470 -> 10k
- R9: value 1k8 -> 10k
- SW1: footprint Button_Switch_THT:SW_Tactile_SPST_Angled_PTS645Vx31-2LFS -> Button_Switch_THT:SW_Tactile_SKHH_Angled
- moved C1 406.5 mm to (-98.0, -60.9)
- moved C1 406.5 mm to (-136.5, -41.2)
- moved C10 406.5 mm to (-94.5, -63.3)
- moved C12 406.5 mm to (-142.3, -37.2)
- moved C13 406.5 mm to (-139.3, -41.2)
- moved C14 406.5 mm to (-139.4, -39.2)
- moved C29 406.5 mm to (-142.2, -39.2)
- moved C8 406.5 mm to (-95.2, -61.3)
- moved C8 406.5 mm to (-145.1, -37.2)
- moved FB3 406.5 mm to (-100.6, -63.1)
- moved FB3 406.5 mm to (-120.8, -39.0)
- moved R29 406.5 mm to (-150.9, -39.2)
- moved R36 406.5 mm to (-145.1, -41.2)
- moved R37 406.5 mm to (-148.0, -37.2)
- moved R38 406.5 mm to (-129.7, -49.9)
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Connections:
- C1 pad 1: Net-(C1-Pad1) -> ENC_A
- C8 pad 1: Net-(C1-Pad1) -> ENC_B
- FB3 pad 1: Net-(C10-Pad1) -> MIC
- FB3 pad 2: Net-(C10-Pad1) -> Net-(FB3-Pad2)
- J2 pad 4: unconnected-(J2-Pad4) -> GND
- R8 pad 1: +5V -> Net-(R36-Pad2)
- R8 pad 2: Net-(C1-Pad1) -> ENC_A
- R9 pad 1: Net-(C1-Pad1) -> Net-(R29-Pad2)
- R9 pad 2: Net-(C10-Pad1) -> ENC_B
- U3 pad 22: BOOT0 -> BTN_F2
- U3 pad 53: R4 -> unconnected-(U3-Pad53)
- U3 pad 54: R3 -> unconnected-(U3-Pad54)
- U3 pad 55: R2 -> unconnected-(U3-Pad55)
- U3 pad 56: R1 -> unconnected-(U3-Pad56)
- U3 pad 57: C1 -> unconnected-(U3-Pad57)
- U3 pad 58: C2 -> unconnected-(U3-Pad58)
- U3 pad 59: C3 -> unconnected-(U3-Pad59)
- U3 pad 60: C4 -> unconnected-(U3-Pad60)
Other:
- board size 99.6 x 43.7 mm -> 95.5 x 107.1 mm
