File: Hardware/KiCAD/HMI/hmi.kicad_sch (KiCad schematic)
At the start: 86 parts, among them J1 PJ-307C, J2 PJ-2282, J3 OLED, J4 Conn_01x30, SW1 SW_Push_45deg, SW10 SW_Push_45deg, SW11 SW_Push_45deg, SW12 SW_Push_45deg, SW13 PTT, SW14 ACZ11BRXE, SW15 SW_Push_45deg, SW16 SW_Push_45deg, SW17 SW_Push_45deg, SW18 SW_Push_45deg, SW19 F1, SW2 SW_Push_45deg, SW20 F2, SW3 SW_Push_45deg, SW4 SW_Push_45deg, SW5 SW_Push_45deg, SW6 SW_Push_45deg, SW7 SW_Push_45deg, SW8 SW_Push_45deg, SW9 SW_Push_45deg, U1 MAX9814, U2 MAX9814

Commit message: Add files via upload
Parts:
- removed C10, C23, C9: 100n, Capacitor_SMD:C_0402_1005Metric, symbol pkl_device:pkl_C_Small
- removed C15: 470n, Capacitor_SMD:C_0402_1005Metric, symbol pkl_device:pkl_C_Small
- removed C16, C24: 2u2, Capacitor_SMD:C_0402_1005Metric, symbol pkl_device:pkl_C_Small
- removed R13: 2k2, Resistor_SMD:R_0402_1005Metric, symbol pkl_device:pkl_R_Small
- removed R14: 0, Resistor_SMD:R_0402_1005Metric, symbol pkl_device:pkl_R_Small
- removed R19: 100k, Resistor_SMD:R_0402_1005Metric, symbol pkl_device:pkl_R_Small
- removed R20: 150k, Resistor_SMD:R_0402_1005Metric, symbol pkl_device:pkl_R_Small
- removed TP2: TP_MIC, TestPoint:TestPoint_Pad_D1.0mm, symbol Connector:TestPoint
- removed TP4: TP_MIC_POST, TestPoint:TestPoint_Pad_D1.0mm, symbol Connector:TestPoint
- removed U2: MAX9814, Package_DFN_QFN:DFN-14-1EP_3x3mm_P0.4mm_EP1.78x2.35mm, symbol Amplifier_Audio:MAX9814
- renumbered C12 to C10, C13 to C11, C14 to C12, C17 to C13, C18 to C14, C19 to C15, C20 to C16, C21 to C17, C22 to C18, C11 to C9, R15 to R13, R16 to R14, R17 to R15, R18 to R16, R21 to R17, R22 to R18, R23 to R19, R24 to R20, TP3 to TP2
Connections:
- no-connect marks 2 -> 5
